File: F3DemoBoard/OshBus_v0.1.sch (KiCad schematic (older format))
At the start: 43 parts, among them J1 Conn_01x02, J2 Conn_01x07, J3 Conn_01x03, J4 Conn_01x06, J5 Conn_02x10_Odd_Even, J6 Conn_01x02, SW1 SW_Push, U1 AZ1117-3.3, U2 AZ1117IH-5.0TRG1, U3 STM32F302K6Ux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

Commit message: Add files via upload
Other:
- note added: "6/24/20\n"
Changed lines of the file:
@@
 	4500 4800 4500 4750
 $Comp
-L power:+3.3V #PWR?
+L power:+3.3V #PWR0147
 U 1 1 5F2D598E
 P 4500 4400
-F 0 "#PWR?" H 4500 4250 50  0001 C CNN
+F 0 "#PWR0147" H 4500 4250 50  0001 C CNN
 F 1 "+3.3V" H 4515 4573 50  0000 C CNN
 F 2 "" H 4500 4400 50  0001 C CNN
@@
 	1    0    0    -1
 $EndComp
+Text Notes 8150 7650 0    39   ~ 0
+6/24/20\n
 $EndSCHEMATC
